Commit message: Add LIDAR and depth camera to robot

File: src/ackermann_robot_description/urdf/ackermann_robot.urdf.xacro (robot description, xacro)
@@ -178,3 +178,98 @@
     </plugin>
   </gazebo>
+  <!--**********************-->
+  <!-- Sensors -->
+  <!--**********************-->
+  <link name="lidar_link">
+    <visual>
+      <geometry>
+        <cylinder length="0.02" radius="0.04"/>
+      </geometry>
+      <origin xyz="0 0 0" rpy="0 0 0"/>
+    </visual>
+    <collision>
+      <geometry>
+        <cylinder length="0.02" radius="0.04"/>
+      </geometry>
+      <origin xyz="0 0 0" rpy="0 0 0"/>
+    </collision>
+    <inertial>
+      <mass value="0.1"/>
+      <inertia ixx="0.001" ixy="0.0" ixz="0.0" iyy="0.001" iyz="0.0" izz="0.001"/>
+    </inertial>
+  </link>
+  <joint name="lidar_joint" type="fixed">
+    <parent link="base_chassis"/>
+    <child link="lidar_link"/>
+    <origin xyz="0 0 ${chassis_height + 0.05}" rpy="0 0 0"/>
+  </joint>
+  <gazebo reference="lidar_link">
+    <sensor name="lidar" type="ray">
+      <pose>0 0 0 0 0 0</pose>
+      <update_rate>10</update_rate>
+      <ray>
+        <scan>
+          <horizontal>
+            <samples>720</samples>
+            <min_angle>-1.5708</min_angle>
+            <max_angle>1.5708</max_angle>
+          </horizontal>
+        </scan>
+        <range>
+          <min>0.1</min>
+          <max>10.0</max>
+          <resolution>0.01</resolution>
+        </range>
+      </ray>
+      <plugin name="gazebo_ros_laser" filename="libgazebo_ros_ray_sensor.so">
+        <topicName>scan</topicName>
+        <frameName>lidar_link</frameName>
+      </plugin>
+    </sensor>
+  </gazebo>
+  <link name="depth_camera_link">
+    <visual>
+      <geometry>
+        <box size="0.05 0.05 0.05"/>
+      </geometry>
+      <origin xyz="0 0 0" rpy="0 0 0"/>
+    </visual>
+    <collision>
+      <geometry>
+        <box size="0.05 0.05 0.05"/>
+      </geometry>
+      <origin xyz="0 0 0" rpy="0 0 0"/>
+    </collision>
+    <inertial>
+      <mass value="0.2"/>
+      <inertia ixx="0.002" ixy="0.0" ixz="0.0" iyy="0.002" iyz="0.0" izz="0.002"/>
+    </inertial>
+  </link>
+  <joint name="depth_camera_joint" type="fixed">
+    <parent link="base_chassis"/>
+    <child link="depth_camera_link"/>
+    <origin xyz="0 0 ${chassis_height + 0.1}" rpy="0 0 0"/>
+  </joint>
+  <gazebo reference="depth_camera_link">
+    <sensor name="depth_camera" type="depth">
+      <pose>0 0 0 0 0 0</pose>
+      <update_rate>30</update_rate>
+      <camera>
+        <horizontal_fov>1.047</horizontal_fov>
+        <image>
+          <width>640</width>
+          <height>480</height>
+          <format>R8G8B8</format>
+        </image>
+        <clip>
+          <near>0.05</near>
+          <far>10.0</far>
+        </clip>
+      </camera>
+      <plugin name="gazebo_ros_depth_camera" filename="libgazebo_ros_depth_camera.so">
+        <topicName>depth/image_raw</topicName>
+        <frameName>depth_camera_link</frameName>
+      </plugin>
+    </sensor>
+  </gazebo>
 </robot>

Commit message: add sensors

File: src/ackermann_robot_description/urdf/ackermann_robot.urdf.xacro (robot description, xacro)
@@ -16,6 +16,27 @@
   <!-- Inertial/Visual/Collision Macros -->
   <!--**********************-->
+    <!-- Define inertial property macros  -->
+  <xacro:macro name="box_inertia" params="m w h d">
+    <inertial>
+      <origin xyz="0 0 0" rpy="${pi/2} 0 ${pi/2}"/>
+      <mass value="${m}"/>
+      <inertia ixx="${(m/12) * (h*h + d*d)}" ixy="0.0" ixz="0.0" iyy="${(m/12) * (w*w + d*d)}" iyz="0.0" izz="${(m/12) * (w*w + h*h)}"/>
+    </inertial>
+  </xacro:macro>
+  <xacro:macro name="cylinder_inertia" params="m r h">
+    <inertial>
+      <origin xyz="0 0 0" rpy="${pi/2} 0 0" />
+      <mass value="${m}"/>
+      <inertia ixx="${(m/12) * (3*r*r + h*h)}" ixy = "0" ixz = "0" iyy="${(m/12) * (3*r*r + h*h)}" iyz = "0" izz="${(m/2) * (r*r)}"/>
+    </inertial>
+  </xacro:macro>
+  <xacro:macro name="sphere_inertia" params="m r">
+    <inertial>
+      <mass value="${m}"/>
+      <inertia ixx="${(2/5) * m * (r*r)}" ixy="0.0" ixz="0.0" iyy="${(2/5) * m * (r*r)}" iyz="0.0" izz="${(2/5) * m * (r*r)}"/>
+    </inertial>
+  </xacro:macro>
   <xacro:macro name="chassis_link" params="prefix">
-    <link name="${prefix}_chassis">
+    <link name="${prefix}_link">
       <visual>
         <geometry>
@@ -74,4 +95,11 @@
   <!--**********************-->
   <xacro:chassis_link prefix="base"/>
+  <!-- Robot Footprint -->
+  <link name="base_footprint"/>
+  <joint name="base_joint" type="fixed">
+    <parent link="base_link"/>
+    <child link="base_footprint"/>
+    <origin xyz="0.0 0.0 ${-(wheel_radius)}" rpy="0 0 0"/>
+  </joint>
   <!--**********************-->
   <!-- Steering Links -->
@@ -96,5 +124,5 @@
   </link>
   <joint name="front_left_steering_joint" type="revolute">
-    <parent link="base_chassis"/>
+    <parent link="base_link"/>
     <child  link="front_left_steering_link"/>
     <origin xyz="${wheelbase/2} ${track_width/2} ${wheel_radius}" rpy="0 0 0"/>
@@ -121,5 +149,5 @@
   </link>
   <joint name="front_right_steering_joint" type="revolute">
-    <parent link="base_chassis"/>
+    <parent link="base_link"/>
     <child  link="front_right_steering_link"/>
     <origin xyz="${wheelbase/2} -${track_width/2} ${wheel_radius}" rpy="0 0 0"/>
@@ -132,5 +160,5 @@
   <xacro:wheel_link
     name="rear_left_wheel"
-    suffix="base_chassis"
+    suffix="base_link"
     pos_x="${-wheelbase/2}"
     pos_y="${track_width/2}"
@@ -139,5 +167,5 @@
   <xacro:wheel_link
     name="rear_right_wheel"
-    suffix="base_chassis"
+    suffix="base_link"
     pos_x="${-wheelbase/2}"
     pos_y="${-track_width/2}"
@@ -181,4 +209,89 @@
   <!-- Sensors -->
   <!--**********************-->
+  <link name="imu_link">
+		<visual>
+		  <geometry>
+		    <box size="0.1 0.1 0.1"/>
+		  </geometry>
+		</visual>
+		<collision>
+		  <geometry>
+		    <box size="0.1 0.1 0.1"/>
+		  </geometry>
+		</collision>
+		<xacro:box_inertia m="0.1" w="0.1" d="0.1" h="0.1"/>
+	</link>
+	<joint name="imu_joint" type="fixed">
+		<parent link="base_link"/>
+		<child link="imu_link"/>
+		<origin xyz="0 0 0.01"/>
+	</joint>
+	 <gazebo reference="imu_link">
+		<sensor name="imu_sensor" type="imu">
+		 <plugin filename="libgazebo_ros_imu_sensor.so" name="imu_plugin">
+		    <ros>
+		      <remapping>~/out:=imu</remapping>
+		    </ros>
+		    <initial_orientation_as_reference>false</initial_orientation_as_reference>
+		  </plugin>
+		  <always_on>true</always_on>
+		  <update_rate>100</update_rate>
+		  <visualize>true</visualize>
+		  <imu>
+		    <angular_velocity>
+		      <x>
+		        <noise type="gaussian">
+		          <mean>0.0</mean>
+		          <stddev>2e-4</stddev>
+		          <bias_mean>0.0000075</bias_mean>
+		          <bias_stddev>0.0000008</bias_stddev>
+		        </noise>
+		      </x>
+		      <y>
+		        <noise type="gaussian">
+		          <mean>0.0</mean>
+		          <stddev>2e-4</stddev>
+		          <bias_mean>0.0000075</bias_mean>
+		          <bias_stddev>0.0000008</bias_stddev>
+		        </noise>
+		      </y>
+		      <z>
+		        <noise type="gaussian">
+		          <mean>0.0</mean>
+		          <stddev>2e-4</stddev>
+		          <bias_mean>0.0000075</bias_mean>
+		          <bias_stddev>0.0000008</bias_stddev>
+		        </noise>
+		      </z>
+		    </angular_velocity>
+		    <linear_acceleration>
+		      <x>
+		        <noise type="gaussian">
+		          <mean>0.0</mean>
+		          <stddev>1.7e-2</stddev>
+		          <bias_mean>0.1</bias_mean>
+		          <bias_stddev>0.001</bias_stddev>
+		        </noise>
+		      </x>
+		      <y>
+		        <noise type="gaussian">
+		          <mean>0.0</mean>
+		          <stddev>1.7e-2</stddev>
+		          <bias_mean>0.1</bias_mean>
+		          <bias_stddev>0.001</bias_stddev>
+		        </noise>
+		      </y>
+		      <z>
+		        <noise type="gaussian">
+		          <mean>0.0</mean>
+		          <stddev>1.7e-2</stddev>
+		          <bias_mean>0.1</bias_mean>
+		          <bias_stddev>0.001</bias_stddev>
+		        </noise>
+		      </z>
+		    </linear_acceleration>
+		  </imu>
+		</sensor>
+	</gazebo>
   <link name="lidar_link">
     <visual>
@@ -200,5 +313,5 @@
   </link>
   <joint name="lidar_joint" type="fixed">
-    <parent link="base_chassis"/>
+    <parent link="base_link"/>
     <child link="lidar_link"/>
     <origin xyz="0 0 ${chassis_height + 0.05}" rpy="0 0 0"/>
@@ -223,6 +336,9 @@
       </ray>
       <plugin name="gazebo_ros_laser" filename="libgazebo_ros_ray_sensor.so">
-        <topicName>scan</topicName>
-        <frameName>lidar_link</frameName>
+		  <ros>
+		    <remapping>~/out:=scan</remapping>
+		  </ros>
+		  <output_type>sensor_msgs/LaserScan</output_type>
+		  <frame_name>lidar_link</frame_name>
       </plugin>
     </sensor>
@@ -247,5 +363,5 @@
   </link>
   <joint name="depth_camera_joint" type="fixed">
-    <parent link="base_chassis"/>
+    <parent link="base_link"/>
     <child link="depth_camera_link"/>
     <origin xyz="0 0 ${chassis_height + 0.1}" rpy="0 0 0"/>
@@ -253,4 +369,5 @@
   <gazebo reference="depth_camera_link">
     <sensor name="depth_camera" type="depth">
+    	<visualize>true</visualize>
       <pose>0 0 0 0 0 0</pose>
       <update_rate>30</update_rate>
@@ -267,7 +384,21 @@
         </clip>
       </camera>
-      <plugin name="gazebo_ros_depth_camera" filename="libgazebo_ros_depth_camera.so">
-        <topicName>depth/image_raw</topicName>
-        <frameName>depth_camera_link</frameName>
+      <plugin name="gazebo_ros_depth_camera" filename="libgazebo_ros_camera.so">
+				<baseline>0.2</baseline>
+				<alwaysOn>true</alwaysOn>
+				<updateRate>0.0</updateRate>
+				<frame_name>camera_depth_frame</frame_name>
+				<pointCloudCutoff>0.5</pointCloudCutoff>
+				<pointCloudCutoffMax>3.0</pointCloudCutoffMax>
+				<distortionK1>0</distortionK1>
+				<distortionK2>0</distortionK2>
+				<distortionK3>0</distortionK3>
+				<distortionT1>0</distortionT1>
+				<distortionT2>0</distortionT2>
+				<CxPrime>0</CxPrime>
+				<Cx>0</Cx>
+				<Cy>0</Cy>
+				<focalLength>0</focalLength>
+				<hackBaseline>0</hackBaseline>
       </plugin>
     </sensor>

Commit message: rviz2 simulation properly set up

File: src/ackermann_robot_description/urdf/ackermann_robot.urdf.xacro (robot description, xacro)
@@ -10,7 +10,21 @@
   <xacro:property name="wheel_radius"  value="0.05"/>
   <xacro:property name="wheel_width"   value="0.03"/>
+  <!-- Ground clearance -->
+  <xacro:property name="ground_clearance" value="${wheel_radius}"/>
   <!-- Axle distances -->
   <xacro:property name="wheelbase"      value="0.4"/>  <!-- distance between front and rear axles -->
   <xacro:property name="track_width"    value="0.3"/>  <!-- distance between left and right wheels -->
+  <!-- Steering link dimensions -->
+  <xacro:property name="steering_link_size" value="0.02"/>
+  <xacro:property name="steering_offset_z" value="0.01"/> <!-- Small offset to prevent collision -->
+  <!-- Sensor placements -->
+  <xacro:property name="imu_height" value="${chassis_height + 0.075}"/>
+  <xacro:property name="lidar_height" value="${chassis_height + 0.05}"/>
+  <xacro:property name="camera_height" value="${chassis_height + 0.15}"/>
+  <!-- Sensor dimensions -->
+  <xacro:property name="imu_size" value="0.05"/>
+  <xacro:property name="lidar_radius" value="0.04"/>
+  <xacro:property name="lidar_height" value="0.02"/>
+  <xacro:property name="camera_size" value="0.05"/>
   <!--**********************-->
   <!-- Inertial/Visual/Collision Macros -->
@@ -46,5 +60,6 @@
           <color rgba="0 0.2 0.8 1.0"/>
         </material>
-        <origin xyz="0 0 ${chassis_height/2}" rpy="0 0 0"/>
+        <!-- The visual origin is at the center of the chassis box -->
+        <origin xyz="0 0 0" rpy="0 0 0"/>
       </visual>
       <collision>
@@ -52,7 +67,8 @@
           <box size="${chassis_length} ${chassis_width} ${chassis_height}"/>
         </geometry>
-        <origin xyz="0 0 ${chassis_height/2}" rpy="0 0 0"/>
+        <origin xyz="0 0 0" rpy="0 0 0"/>
       </collision>
       <inertial>
+        <origin xyz="0 0 0" rpy="0 0 0"/>
         <mass value="5.0"/>
         <inertia ixx="0.1" ixy="0.0" ixz="0.0" iyy="0.1" iyz="0.0" izz="0.1"/>
@@ -79,4 +95,5 @@
       </collision>
       <inertial>
+        <origin xyz="0 0 0" rpy="1.5708 0 0"/>
         <mass value="0.5"/>
         <inertia ixx="0.001" ixy="0.0" ixz="0.0" iyy="0.001" iyz="0.0" izz="0.0005"/>
@@ -89,4 +106,6 @@
       <origin xyz="${pos_x} ${pos_y} ${pos_z}" rpy="0 0 0"/>
       <axis   xyz="0 1 0"/>
+      <!-- Add dynamics properties for better simulation -->
+      <dynamics damping="0.01" friction="0.1"/>
     </joint>
   </xacro:macro>
@@ -94,11 +113,30 @@
   <!-- Chassis -->
   <!--**********************-->
+  <!-- Base footprint is a virtual frame at the ground directly beneath the robot's center -->
+  <link name="base_footprint">
+    <!-- Visual marker only - no collision or significant mass -->
+    <visual>
+      <geometry>
+        <sphere radius="0.001"/>
+      </geometry>
+      <material name="Green">
+        <color rgba="0 1 0 1.0"/>
+      </material>
+    </visual>
+    <!-- Remove collision to eliminate physical interaction with ground -->
+    <!-- Minimal inertia to avoid dynamics issues -->
+    <inertial>
+      <mass value="0.0000001"/>
+      <inertia ixx="0.0" ixy="0.0" ixz="0.0" iyy="0.0" iyz="0.0" izz="0.0"/>
+    </inertial>
+  </link>
+  <!-- Create the chassis -->
   <xacro:chassis_link prefix="base"/>
-  <!-- Robot Footprint -->
-  <link name="base_footprint"/>
+  <!-- Connect base_footprint to base_link with fixed joint but no physical constraints -->
   <joint name="base_joint" type="fixed">
-    <parent link="base_link"/>
-    <child link="base_footprint"/>
-    <origin xyz="0.0 0.0 ${-(wheel_radius)}" rpy="0 0 0"/>
+    <parent link="base_footprint"/>
+    <child link="base_link"/>
+    <!-- Position base_link at the 3D center of the robot, above the footprint -->
+    <origin xyz="0 0 ${ground_clearance + chassis_height/2}" rpy="0 0 0"/>
   </joint>
   <!--**********************-->
@@ -108,11 +146,14 @@
     <visual>
       <geometry>
-        <box size="0.02 0.02 0.02"/>
-      </geometry>
-      <origin xyz="0 0 0" rpy="0 0 0"/>
+        <box size="${steering_link_size} ${steering_link_size} ${steering_link_size}"/>
+      </geometry>
+      <origin xyz="0 0 0" rpy="0 0 0"/>
+      <material name="Gray">
+        <color rgba="0.5 0.5 0.5 1.0"/>
+      </material>
     </visual>
     <collision>
       <geometry>
-        <box size="0.02 0.02 0.02"/>
+        <box size="${steering_link_size} ${steering_link_size} ${steering_link_size}"/>
       </geometry>
       <origin xyz="0 0 0" rpy="0 0 0"/>
@@ -126,5 +167,6 @@
     <parent link="base_link"/>
     <child  link="front_left_steering_link"/>
-    <origin xyz="${wheelbase/2} ${track_width/2} ${wheel_radius}" rpy="0 0 0"/>
+    <!-- Adjust the steering joint position relative to the center of base_link -->
+    <origin xyz="${wheelbase/2} ${track_width/2} 0" rpy="0 0 0"/>
     <axis  xyz="0 0 1"/>
     <limit lower="-0.785" upper="0.785" effort="5.0" velocity="5.0"/>
@@ -133,11 +175,14 @@
     <visual>
       <geometry>
-        <box size="0.02 0.02 0.02"/>
-      </geometry>
-      <origin xyz="0 0 0" rpy="0 0 0"/>
+        <box size="${steering_link_size} ${steering_link_size} ${steering_link_size}"/>
+      </geometry>
+      <origin xyz="0 0 0" rpy="0 0 0"/>
+      <material name="Gray">
+        <color rgba="0.5 0.5 0.5 1.0"/>
+      </material>
     </visual>
     <collision>
       <geometry>
-        <box size="0.02 0.02 0.02"/>
+        <box size="${steering_link_size} ${steering_link_size} ${steering_link_size}"/>
       </geometry>
       <origin xyz="0 0 0" rpy="0 0 0"/>
@@ -151,5 +196,6 @@
     <parent link="base_link"/>
     <child  link="front_right_steering_link"/>
-    <origin xyz="${wheelbase/2} -${track_width/2} ${wheel_radius}" rpy="0 0 0"/>
+    <!-- Adjust the steering joint position relative to the center of base_link -->
+    <origin xyz="${wheelbase/2} -${track_width/2} 0" rpy="0 0 0"/>
     <axis  xyz="0 0 1"/>
     <limit lower="-0.785" upper="0.785" effort="5.0" velocity="5.0"/>
@@ -162,6 +208,6 @@
     suffix="base_link"
     pos_x="${-wheelbase/2}"
-    pos_y="${track_width/2}"
-    pos_z="${wheel_radius}"
+    pos_y="${track_width/2 + wheel_width/2 + 0.01}"
+    pos_z="${-chassis_height/2}"
   />
   <xacro:wheel_link
@@ -169,12 +215,24 @@
     suffix="base_link"
     pos_x="${-wheelbase/2}"
-    pos_y="${-track_width/2}"
-    pos_z="${wheel_radius}"
+    pos_y="${-track_width/2 - wheel_width/2 - 0.01}"
+    pos_z="${-chassis_height/2}"
   />
   <!--**********************-->
   <!-- Front Wheels (mounted) -->
   <!--**********************-->
-  <xacro:wheel_link name="front_left_wheel" suffix="front_left_steering_link" pos_x="0" pos_y="0" pos_z="0"/>
-  <xacro:wheel_link name="front_right_wheel" suffix="front_right_steering_link" pos_x="0" pos_y="0" pos_z="0"/>
+  <xacro:wheel_link
+    name="front_left_wheel"
+    suffix="front_left_steering_link"
+    pos_x="0"
+    pos_y="${wheel_width/2 + 0.01}"
+    pos_z="${-chassis_height/2}"
+  />
+  <xacro:wheel_link
+    name="front_right_wheel"
+    suffix="front_right_steering_link"
+    pos_x="0"
+    pos_y="${-wheel_width/2 - 0.01}"
+    pos_z="${-chassis_height/2}"
+  />
   <!--**********************-->
   <!-- ros2_control Transmissions -->
@@ -187,16 +245,20 @@
       <command_interface name="velocity"/>
       <state_interface   name="velocity"/>
+      <state_interface   name="position"/>
     </joint>
     <joint name="rear_right_wheel_joint">
       <command_interface name="velocity"/>
       <state_interface   name="velocity"/>
+      <state_interface   name="position"/>
     </joint>
     <joint name="front_left_steering_joint">
       <command_interface name="position"/>
       <state_interface   name="position"/>
+      <state_interface   name="velocity"/>
     </joint>
     <joint name="front_right_steering_joint">
       <command_interface name="position"/>
       <state_interface   name="position"/>
+      <state_interface   name="velocity"/>
     </joint>
   </ros2_control>
@@ -210,22 +272,28 @@
   <!--**********************-->
   <link name="imu_link">
-		<visual>
-		  <geometry>
-		    <box size="0.1 0.1 0.1"/>
-		  </geometry>
-		</visual>
-		<collision>
-		  <geometry>
-		    <box size="0.1 0.1 0.1"/>
-		  </geometry>
-		</collision>
-		<xacro:box_inertia m="0.1" w="0.1" d="0.1" h="0.1"/>
-	</link>
-	<joint name="imu_joint" type="fixed">
-		<parent link="base_link"/>
-		<child link="imu_link"/>
-		<origin xyz="0 0 0.01"/>
-	</joint>
-	 <gazebo reference="imu_link">
+    <visual>
+      <geometry>
+        <box size="${imu_size} ${imu_size} ${imu_size}"/>
+      </geometry>
+      <material name="Red">
+        <color rgba="0.8 0.1 0.1 1.0"/>
+      </material>
+      <origin xyz="0 0 0" rpy="0 0 0"/>
+    </visual>
+    <collision>
+      <geometry>
+        <box size="${imu_size} ${imu_size} ${imu_size}"/>
+      </geometry>
+      <origin xyz="0 0 0" rpy="0 0 0"/>
+    </collision>
+    <xacro:box_inertia m="0.1" w="${imu_size}" d="${imu_size}" h="${imu_size}"/>
+  </link>
+  <joint name="imu_joint" type="fixed">
+    <parent link="base_link"/>
+    <child link="imu_link"/>
+    <!-- Adjust the position relative to the center of base_link -->
+    <origin xyz="${wheelbase/4} 0 ${chassis_height/2 + imu_size/2}" rpy="0 0 0"/>
+  </joint>
+  <gazebo reference="imu_link">
 		<sensor name="imu_sensor" type="imu">
 		 <plugin filename="libgazebo_ros_imu_sensor.so" name="imu_plugin">
@@ -297,11 +365,14 @@
     <visual>
       <geometry>
-        <cylinder length="0.02" radius="0.04"/>
-      </geometry>
+        <cylinder length="${lidar_height}" radius="${lidar_radius}"/>
+      </geometry>
+      <material name="Green">
+        <color rgba="0.1 0.8 0.1 1.0"/>
+      </material>
       <origin xyz="0 0 0" rpy="0 0 0"/>
     </visual>
     <collision>
       <geometry>
-        <cylinder length="0.02" radius="0.04"/>
+        <cylinder length="${lidar_height}" radius="${lidar_radius}"/>
       </geometry>
       <origin xyz="0 0 0" rpy="0 0 0"/>
@@ -309,4 +380,5 @@
     <inertial>
       <mass value="0.1"/>
+      <origin xyz="0 0 0" rpy="0 0 0"/>
       <inertia ixx="0.001" ixy="0.0" ixz="0.0" iyy="0.001" iyz="0.0" izz="0.001"/>
     </inertial>
@@ -315,5 +387,6 @@
     <parent link="base_link"/>
     <child link="lidar_link"/>
-    <origin xyz="0 0 ${chassis_height + 0.05}" rpy="0 0 0"/>
+    <!-- Adjust the position relative to the center of base_link -->
+    <origin xyz="0 0 ${chassis_height/2 + lidar_height/2}" rpy="0 0 0"/>
   </joint>
   <gazebo reference="lidar_link">
@@ -347,11 +420,14 @@
     <visual>
       <geometry>
-        <box size="0.05 0.05 0.05"/>
-      </geometry>
+        <box size="${camera_size} ${camera_size} ${camera_size}"/>
+      </geometry>
+      <material name="Yellow">
+        <color rgba="0.8 0.8 0.1 1.0"/>
+      </material>
       <origin xyz="0 0 0" rpy="0 0 0"/>
     </visual>
     <collision>
       <geometry>
-        <box size="0.05 0.05 0.05"/>
+        <box size="${camera_size} ${camera_size} ${camera_size}"/>
       </geometry>
       <origin xyz="0 0 0" rpy="0 0 0"/>
@@ -359,4 +435,5 @@
     <inertial>
       <mass value="0.2"/>
+      <origin xyz="0 0 0" rpy="0 0 0"/>
       <inertia ixx="0.002" ixy="0.0" ixz="0.0" iyy="0.002" iyz="0.0" izz="0.002"/>
     </inertial>
@@ -365,5 +442,6 @@
     <parent link="base_link"/>
     <child link="depth_camera_link"/>
-    <origin xyz="0 0 ${chassis_height + 0.1}" rpy="0 0 0"/>
+    <!-- Adjust the position relative to the center of base_link -->
+    <origin xyz="${wheelbase/3} 0 ${chassis_height/2 + camera_size/2 + 0.05}" rpy="0 0 0"/>
   </joint>
   <gazebo reference="depth_camera_link">
