Commit message: complete proj

File: src/ackermann_robot_description/urdf/ackermann_robot.urdf.xacro (robot description, xacro)
@@ -1,35 +1,491 @@
 <?xml version="1.0"?>
 <robot xmlns:xacro="http://ros.org/wiki/xacro" name="ackermann_robot">
-  <!-- Depth Camera Sensor -->
-  <link name="depth_camera_link">
-    <inertial>
-      <origin xyz="0 0 0" rpy="0 0 0"/>
-      <mass value="0.035"/>
-      <inertia ixx="0.001"  ixy="0"  ixz="0" iyy="0.001" iyz="0" izz="0.001" />
-    </inertial>
-    <collision>
-      <origin xyz="0 0 0" rpy="0 0 0"/>
-      <geometry>
-        <box size="0.015 0.130 0.022"/>
-      </geometry>
-    </collision>
-    <visual>
-      <origin xyz="0 0 0" rpy="0 0 0"/>
-      <geometry>
-        <box size="0.015 0.130 0.022"/>
-      </geometry>
-      <material name="Yellow">
-        <color rgba="0.8 0.8 0.2 1.0"/>
-      </material>
-    </visual>
-  </link>
-  <joint name="depth_camera_joint" type="fixed">
-    <parent link="base_link"/>
-    <child link="depth_camera_link"/>
-    <origin xyz="0.215 0 0.05" rpy="0 0 0"/>
-  </joint>
-  <link name="depth_camera_frame"/>
-  <joint name="depth_camera_frame_joint" type="fixed">
-    <origin xyz="0 0 0" rpy="${-pi/2} 0 ${-pi/2}"/>
-    <parent link="depth_camera_link"/>
-    <child link="depth_camera_frame"/>
+    <!--**********************-->
+    <!-- Define Macros/Properties -->
+    <!--**********************-->
+    <xacro:property name="chassis_length" value="0.6"/>
+    <xacro:property name="chassis_width" value="0.4"/>
+    <xacro:property name="chassis_height" value="0.1"/>
+    <!-- Wheel dimensions -->
+    <xacro:property name="wheel_radius" value="0.05"/>
+    <xacro:property name="wheel_width" value="0.03"/>
+    <!-- Ground clearance -->
+    <xacro:property name="ground_clearance" value="${wheel_radius}"/>
+    <!-- Axle distances -->
+    <xacro:property name="wheelbase" value="0.4"/>  <!-- distance between front and rear axles -->
+    <xacro:property name="track_width" value="0.3"/>  <!-- distance between left and right wheels -->
+    <!-- Steering link dimensions -->
+    <xacro:property name="steering_link_size" value="0.02"/>
+    <xacro:property name="steering_offset_z" value="0.01"/> <!-- Small offset to prevent collision -->
+    <!-- Sensor placements -->
+    <xacro:property name="imu_height" value="${chassis_height + 0.075}"/>
+    <xacro:property name="lidar_height" value="${chassis_height + 0.05}"/>
+    <xacro:property name="camera_height" value="${chassis_height + 0.15}"/>
+    <!-- Sensor dimensions -->
+    <xacro:property name="imu_size" value="0.05"/>
+    <xacro:property name="lidar_radius" value="0.04"/>
+    <xacro:property name="lidar_height" value="0.02"/>
+    <xacro:property name="camera_size" value="0.05"/>
+    <!--**********************-->
+    <!-- Inertial/Visual/Collision Macros -->
+    <!--**********************-->
+    <!-- Define inertial property macros  -->
+    <xacro:macro name="box_inertia" params="m w h d">
+        <inertial>
+            <origin xyz="0 0 0" rpy="${pi/2} 0 ${pi/2}"/>
+            <mass value="${m}"/>
+            <inertia ixx="${(m/12) * (h*h + d*d)}" ixy="0.0" ixz="0.0" iyy="${(m/12) * (w*w + d*d)}" iyz="0.0"
+                     izz="${(m/12) * (w*w + h*h)}"/>
+        </inertial>
+    </xacro:macro>
+    <xacro:macro name="cylinder_inertia" params="m r h">
+        <inertial>
+            <origin xyz="0 0 0" rpy="${pi/2} 0 0"/>
+            <mass value="${m}"/>
+            <inertia ixx="${(m/12) * (3*r*r + h*h)}" ixy="0" ixz="0" iyy="${(m/12) * (3*r*r + h*h)}" iyz="0"
+                     izz="${(m/2) * (r*r)}"/>
+        </inertial>
+    </xacro:macro>
+    <xacro:macro name="sphere_inertia" params="m r">
+        <inertial>
+            <mass value="${m}"/>
+            <inertia ixx="${(2/5) * m * (r*r)}" ixy="0.0" ixz="0.0" iyy="${(2/5) * m * (r*r)}" iyz="0.0"
+                     izz="${(2/5) * m * (r*r)}"/>
+        </inertial>
+    </xacro:macro>
+    <xacro:macro name="chassis_link" params="prefix">
+        <link name="${prefix}_link">
+            <visual>
+                <geometry>
+                    <box size="${chassis_length} ${chassis_width} ${chassis_height}"/>
+                </geometry>
+                <material name="Blue">
+                    <color rgba="0 0.2 0.8 1.0"/>
+                </material>
+                <!-- The visual origin is at the center of the chassis box -->
+                <origin xyz="0 0 0" rpy="0 0 0"/>
+            </visual>
+            <collision>
+                <geometry>
+                    <box size="${chassis_length} ${chassis_width} ${chassis_height}"/>
+                </geometry>
+                <origin xyz="0 0 0" rpy="0 0 0"/>
+            </collision>
+            <inertial>
+                <origin xyz="0 0 0" rpy="0 0 0"/>
+                <mass value="5.0"/>
+                <inertia ixx="0.1" ixy="0.0" ixz="0.0" iyy="0.1" iyz="0.0" izz="0.1"/>
+            </inertial>
+        </link>
+    </xacro:macro>
+    <xacro:macro name="wheel_link" params="name suffix pos_x pos_y pos_z">
+        <link name="${name}">
+            <visual>
+                <!-- Rotate cylinder so its axis aligns with joint axis -->
+                <origin xyz="0 0 0" rpy="1.5708 0 0"/>
+                <geometry>
+                    <cylinder length="${wheel_width}" radius="${wheel_radius}"/>
+                </geometry>
+                <material name="Black">
+                    <color rgba="0 0 0 1.0"/>
+                </material>
+            </visual>
+            <collision>
+                <origin xyz="0 0 0" rpy="1.5708 0 0"/>
+                <geometry>
+                    <cylinder length="${wheel_width}" radius="${wheel_radius}"/>
+                </geometry>
+            </collision>
+            <inertial>
+                <origin xyz="0 0 0" rpy="1.5708 0 0"/>
+                <mass value="0.5"/>
+                <inertia ixx="0.001" ixy="0.0" ixz="0.0" iyy="0.001" iyz="0.0" izz="0.0005"/>
+            </inertial>
+        </link>
+        <!-- Joint connecting wheel to chassis or steering link -->
+        <joint name="${name}_joint" type="continuous">
+            <parent link="${suffix}"/>
+            <child link="${name}"/>
+            <origin xyz="${pos_x} ${pos_y} ${pos_z}" rpy="0 0 0"/>
+            <axis xyz="0 1 0"/>
+            <!-- Add dynamics properties for better simulation -->
+            <dynamics damping="0.01" friction="0.1"/>
+        </joint>
+    </xacro:macro>
+    <!--**********************-->
+    <!-- Chassis -->
+    <!--**********************-->
+    <!-- Base footprint is a virtual frame at the ground directly beneath the robot's center -->
+    <link name="base_footprint"/>
+    <joint name="base_footprint_joint" type="fixed">
+        <parent link="base_footprint"/>
+        <child link="base_link"/>
+        <origin xyz="0 0 ${wheel_radius}" rpy="0 0 0"/>
+    </joint>
+    <!-- Create the chassis -->
+    <xacro:chassis_link prefix="base"/>
+    <!--**********************-->
+    <!-- Steering Links -->
+    <!--**********************-->
+    <link name="front_left_steering_link">
+        <visual>
+            <geometry>
+                <box size="${steering_link_size} ${steering_link_size} ${steering_link_size}"/>
+            </geometry>
+            <origin xyz="0 0 0" rpy="0 0 0"/>
+            <material name="Gray">
+                <color rgba="0.5 0.5 0.5 1.0"/>
+            </material>
+        </visual>
+        <collision>
+            <geometry>
+                <box size="${steering_link_size} ${steering_link_size} ${steering_link_size}"/>
+            </geometry>
+            <origin xyz="0 0 0" rpy="0 0 0"/>
+        </collision>
+        <inertial>
+            <mass value="0.1"/>
+            <inertia ixx="0.0001" ixy="0.0" ixz="0.0" iyy="0.0001" iyz="0.0" izz="0.0001"/>
+        </inertial>
+    </link>
+    <joint name="front_left_steering_joint" type="revolute">
+        <parent link="base_link"/>
+        <child link="front_left_steering_link"/>
+        <!-- Adjust the steering joint position relative to the center of base_link -->
+        <origin xyz="${wheelbase/2} ${track_width/2} 0" rpy="0 0 0"/>
+        <axis xyz="0 0 1"/>
+        <limit lower="-0.785" upper="0.785" effort="5.0" velocity="5.0"/>
+    </joint>
+    <link name="front_right_steering_link">
+        <visual>
+            <geometry>
+                <box size="${steering_link_size} ${steering_link_size} ${steering_link_size}"/>
+            </geometry>
+            <origin xyz="0 0 0" rpy="0 0 0"/>
+            <material name="Gray">
+                <color rgba="0.5 0.5 0.5 1.0"/>
+            </material>
+        </visual>
+        <collision>
+            <geometry>
+                <box size="${steering_link_size} ${steering_link_size} ${steering_link_size}"/>
+            </geometry>
+            <origin xyz="0 0 0" rpy="0 0 0"/>
+        </collision>
+        <inertial>
+            <mass value="0.1"/>
+            <inertia ixx="0.0001" ixy="0.0" ixz="0.0" iyy="0.0001" iyz="0.0" izz="0.0001"/>
+        </inertial>
+    </link>
+    <joint name="front_right_steering_joint" type="revolute">
+        <parent link="base_link"/>
+        <child link="front_right_steering_link"/>
+        <!-- Adjust the steering joint position relative to the center of base_link -->
+        <origin xyz="${wheelbase/2} -${track_width/2} 0" rpy="0 0 0"/>
+        <axis xyz="0 0 1"/>
+        <limit lower="-0.785" upper="0.785" effort="5.0" velocity="5.0"/>
+    </joint>
+    <!--**********************-->
+    <!-- Rear Wheels (driven) -->
+    <!--**********************-->
+    <xacro:wheel_link
+            name="rear_left_wheel"
+            suffix="base_link"
+            pos_x="${-wheelbase/2}"
+            pos_y="${track_width/2 + wheel_width/2 + 0.01}"
+            pos_z="${-chassis_height/2}"
+    />
+    <xacro:wheel_link
+            name="rear_right_wheel"
+            suffix="base_link"
+            pos_x="${-wheelbase/2}"
+            pos_y="${-track_width/2 - wheel_width/2 - 0.01}"
+            pos_z="${-chassis_height/2}"
+    />
+    <!--**********************-->
+    <!-- Front Wheels (mounted) -->
+    <!--**********************-->
+    <xacro:wheel_link
+            name="front_left_wheel"
+            suffix="front_left_steering_link"
+            pos_x="0"
+            pos_y="${wheel_width/2 + 0.01}"
+            pos_z="${-chassis_height/2}"
+    />
+    <xacro:wheel_link
+            name="front_right_wheel"
+            suffix="front_right_steering_link"
+            pos_x="0"
+            pos_y="${-wheel_width/2 - 0.01}"
+            pos_z="${-chassis_height/2}"
+    />
+    <!--**********************-->
+    <!-- ros2_control Transmissions -->
+    <!--**********************-->
+    <ros2_control name="Ackermann" type="system">
+        <hardware>
+            <plugin>gazebo_ros2_control/GazeboSystem</plugin>
+        </hardware>
+        <joint name="rear_left_wheel_joint">
+            <command_interface name="velocity">
+                <param name="min">-10</param>
+                <param name="max">10</param>
+            </command_interface>
+            <state_interface name="velocity"/>
+            <state_interface name="position"/>
+        </joint>
+        <joint name="rear_right_wheel_joint">
+            <command_interface name="velocity">
+                <param name="min">-10</param>
+                <param name="max">10</param>
+            </command_interface>
+            <state_interface name="velocity"/>
+            <state_interface name="position"/>
+        </joint>
+        <joint name="front_left_steering_joint">
+            <command_interface name="position">
+                <param name="min">-0.785</param>
+                <param name="max">0.785</param>
+            </command_interface>
+            <state_interface name="position"/>
+            <state_interface name="velocity"/>
+        </joint>
+        <joint name="front_right_steering_joint">
+            <command_interface name="position">
+                <param name="min">-0.785</param>
+                <param name="max">0.785</param>
+            </command_interface>
+            <state_interface name="position"/>
+            <state_interface name="velocity"/>
+        </joint>
+    </ros2_control>
+    <gazebo>
+        <plugin name="gazebo_ros2_control" filename="libgazebo_ros2_control.so">
+            <parameters>$(find ackermann_robot_description)/config/ros2_control.yaml</parameters>
+            <robot_param>robot_description</robot_param>
+            <robot_param_node>robot_state_publisher</robot_param_node>
+        </plugin>
+    </gazebo>
+    <!--**********************-->
+    <!-- Sensors -->
+    <!--**********************-->
+    <!-- LiDAR Sensor -->
+    <link name="lidar_link">
+        <inertial>
+            <origin xyz="0 0 0" rpy="0 0 0"/>
+            <mass value="0.125"/>
+            <inertia ixx="0.001" ixy="0" ixz="0" iyy="0.001" iyz="0" izz="0.001"/>
+        </inertial>
+        <collision>
+            <origin xyz="0 0 0" rpy="0 0 0"/>
+            <geometry>
+                <cylinder radius="0.0508" length="0.055"/>
+            </geometry>
+        </collision>
+        <visual>
+            <origin xyz="0 0 0" rpy="0 0 0"/>
+            <geometry>
+                <cylinder radius="0.0508" length="0.055"/>
+            </geometry>
+        </visual>
+    </link>
+    <joint name="lidar_joint" type="fixed">
+        <parent link="base_link"/>
+        <child link="lidar_link"/>
+        <!-- Adjust the position relative to the center of base_link -->
+        <origin xyz="0 0 ${chassis_height/2 + lidar_height/2}" rpy="0 0 0"/>
+    </joint>
+    <gazebo reference="lidar_link">
+        <sensor name="lidar" type="ray">
+            <pose>0 0 0 0 0 0</pose>
+            <update_rate>10</update_rate>
+            <ray>
+                <scan>
+                    <horizontal>
+                        <samples>360</samples>
+                        <resolution>1.000000</resolution>
+                        <min_angle>-0.000000</min_angle>
+                        <max_angle>6.280000</max_angle>
+                    </horizontal>
+                </scan>
+                <range>
+                    <min>0.1</min>
+                    <max>3.5</max>
+                    <resolution>0.015000</resolution>
+                </range>
+                <noise>
+                    <type>gaussian</type>
+                    <mean>0.0</mean>
+                    <stddev>0.01</stddev>
+                </noise>
+            </ray>
+            <plugin name="gazebo_ros_laser" filename="libgazebo_ros_ray_sensor.so">
+                <ros>
+                    <remapping>~/out:=scan</remapping>
+                </ros>
+                <output_type>sensor_msgs/LaserScan</output_type>
+                <frame_name>lidar_link</frame_name>
+            </plugin>
+        </sensor>
+    </gazebo>
+    <!-- Depth Camera Sensor -->
+    <link name="depth_camera_link">
+        <inertial>
+            <origin xyz="0 0 0" rpy="0 0 0"/>
+            <mass value="0.1"/>
+            <inertia ixx="0.0001" ixy="0" ixz="0" iyy="0.0001" iyz="0" izz="0.0001"/>
+        </inertial>
+        <collision>
+            <origin xyz="0 0 0" rpy="0 0 0"/>
+            <geometry>
+                <box size="${camera_size} ${camera_size} ${camera_size/2}"/>
+            </geometry>
+        </collision>
+        <visual>
+            <origin xyz="0 0 0" rpy="0 0 0"/>
+            <geometry>
+                <box size="${camera_size} ${camera_size} ${camera_size/2}"/>
+            </geometry>
+            <material name="Yellow">
+                <color rgba="0.8 0.8 0.2 1.0"/>
+            </material>
+        </visual>
+    </link>
+    <joint name="depth_camera_joint" type="fixed">
+        <parent link="base_link"/>
+        <child link="depth_camera_link"/>
+        <!-- Position the depth camera at the front of the robot with a height offset -->
+        <origin xyz="${chassis_length/2} 0 ${chassis_height/2 - camera_height/4}" rpy="0 0 0"/>
+    </joint>
+    <gazebo reference="depth_camera_link">
+        <sensor name="depth_camera" type="depth">
+            <update_rate>30.0</update_rate>
+            <camera>
+                <horizontal_fov>1.047198</horizontal_fov>
+                <image>
+                    <width>640</width>
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